Commit message: modified urdf to represent actual robot pose in gazebo

File: kortex_description/robots/kortex_robot.xacro (robot description, xacro)
@@ -22,5 +22,5 @@
                 <child link="${prefix}base_link" />
                 <parent link="world" />
-                <origin xyz="0 0 0" rpy="0 0 0" />
+                <origin xyz="0 0 1.02" rpy="0 0 0" />
             </joint>
         </xacro:if>
