Commit message: updated the model with shorter loop handle

File: kortex_description/grippers/loop_handle/urdf/loop_handle.xacro (robot description, xacro)
@@ -6,9 +6,9 @@
         <parent link="${parent}"/>
         <child link="${prefix}long_handle_base_link"/>
-        <origin rpy="0.0 0.0 0" xyz="0.0 0.0 0.028"/>
+        <origin rpy="0.0 0.0 0" xyz="0.0 0.0 0.0"/>
     </joint>
     <link name="${prefix}long_handle_base_link">
       <inertial>
-        <origin xyz="8.625E-08 -4.6583E-06 0.03145" rpy="0 0 0" />
+        <origin xyz="8.625E-08 -4.6583E-06 0" rpy="0 0 0" />
         <mass value="0.22652" />
         <inertia ixx="0.00020005" ixy="-4.2442E-10" ixz="-2.9069E-10" iyy="0.00017832" iyz="-3.4402E-08" izz="0.00013478" />
@@ -19,5 +19,6 @@
           <!-- The DAE file doesn't show well in Gazebo so we're using the STL instead -->
           <!-- <mesh filename="package://kortex_description/grippers/robotiq_2f_85/meshes/visual/robotiq_arg2f_85_base_link.dae" scale="0.001 0.001 0.001"/> -->
-          <mesh scale="0.001 0.001 0.001" filename="package://kortex_description/grippers/loop_handle/meshes/visual/long_loop_handle.stl" />
+          <!-- <mesh scale="0.001 0.001 0.001" filename="package://kortex_description/grippers/loop_handle/meshes/visual/long_loop_handle.stl" /> -->
+          <mesh filename="package://kortex_description/grippers/loop_handle/meshes/visual/short_loop_handle.obj"/>
         </geometry>
         <material name="">
@@ -28,5 +29,6 @@
         <origin xyz="0 0 0" rpy="0 0 0" />
         <geometry>
-           <mesh scale="0.001 0.001 0.001" filename="package://kortex_description/grippers/loop_handle/meshes/collision/long_loop_handle.stl" />
+          <mesh filename="package://kortex_description/grippers/loop_handle/meshes/visual/short_loop_handle.obj"/>
+          <!-- <mesh scale="0.001 0.001 0.001" filename="package://kortex_description/grippers/loop_handle/meshes/collision/long_loop_handle.stl" /> -->
         </geometry>
       </collision>

File: kortex_description/grippers/loop_handle/urdf/loop_handle_model_macro.xacro (robot description, xacro)
@@ -7,5 +7,5 @@
     <link name="${prefix}tool_frame"/>
     <joint name="${prefix}tool_frame_joint" type="fixed">
-        <origin xyz="0 0 0.209" rpy="0 0 0" />
+        <origin xyz="0 0 0.164" rpy="0 0 0" />
         <parent link="${parent}" />
         <child link="${prefix}tool_frame" />
@@ -14,10 +14,4 @@
     <!-- Gripper description -->
     <xacro:loop_handle_base_link prefix="${prefix}" parent="${parent}"/>
-    <!-- <xacro:finger_links prefix="${prefix}" fingerprefix="left" stroke="85"/>
-    <xacro:finger_links prefix="${prefix}" fingerprefix="right" stroke="85"/>
-    <xacro:finger_joint prefix="${prefix}"/>
-    <xacro:right_outer_knuckle_joint prefix="${prefix}"/> -->
-    <!-- Transmissions are loaded in the generic kortex xacro when simulation is enabled -->
-    <!-- <xacro:robotiq_arg2f_transmission prefix="${prefix}"/> -->
   </xacro:macro>
 </robot>
